Commit message: Updated ROS URDF to C6.1

File: Visualization/ROS/Space_Gripper_URDF.urdf (robot description, URDF)
Before this commit: robot Space_Gripper_URDF, 13 links, 12 joints
Links:
- link finger_link13_1: mass 0.061687 -> 0.165174
- link finger_link23_1: mass 0.061687 -> 0.165174
- link finger_link33_1: mass 0.061687 -> 0.165174
Joints:
- joint finger_joint_1_3: axis -0.0 -0.01 -0.0 -> 0.0 0.01 0.0; limit lower=-1.570796 upper=0.0 effort=100 velocity=100 -> lower=-1.570796 upper=1.570796 effort=100 velocity=100
- joint finger_joint_2_3: limit lower=0.0 upper=1.570796 effort=100 velocity=100 -> lower=-1.570796 upper=1.570796 effort=100 velocity=100
- joint finger_joint_3_3: axis -0.00866 0.005 -0.0 -> 0.00866 -0.005 0.0; limit lower=-1.570796 upper=0.0 effort=100 velocity=100 -> lower=-1.570796 upper=1.570796 effort=100 velocity=100
