Commit message: Updated URDF and Meshes for PyBullet

File: Visualization/PyBullet/Space_Gripper_URDF.urdf (robot description, URDF)
Before this commit: robot Space_Gripper_URDF, 13 links, 12 joints
Links:
- removed link finger_link111
- removed link finger_link121
- removed link finger_link131
- removed link finger_link211
- removed link finger_link221
- removed link finger_link231
- removed link finger_link311
- removed link finger_link321
- removed link finger_link331
- removed link palm_link11
- removed link palm_link21
- removed link palm_link31
- added link finger_link11_1, mass 0.058758; collision mesh filename=package://fusion2urdf/Space_Gripper_URDF/bin_stl/finger_lin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; visual mesh filename=package://fusion2urdf/Space_Gripper_URDF/bin_stl/finger_lin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
- added link finger_link12_1, mass 0.058758; collision mesh filename=package://fusion2urdf/Space_Gripper_URDF/bin_stl/finger_lin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; visual mesh filename=package://fusion2urdf/Space_Gripper_URDF/bin_stl/finger_lin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
- added link finger_link13_1, mass 0.165174; collision mesh filename=package://fusion2urdf/Space_Gripper_URDF/bin_stl/finger_lin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; visual mesh filename=package://fusion2urdf/Space_Gripper_URDF/bin_stl/finger_lin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
- added link finger_link21_1, mass 0.058758; collision mesh filename=package://fusion2urdf/Space_Gripper_URDF/bin_stl/finger_lin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; visual mesh filename=package://fusion2urdf/Space_Gripper_URDF/bin_stl/finger_lin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
- added link finger_link22_1, mass 0.058758; collision mesh filename=package://fusion2urdf/Space_Gripper_URDF/bin_stl/finger_lin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; visual mesh filename=package://fusion2urdf/Space_Gripper_URDF/bin_stl/finger_lin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
- added link finger_link23_1, mass 0.165174; collision mesh filename=package://fusion2urdf/Space_Gripper_URDF/bin_stl/finger_lin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; visual mesh filename=package://fusion2urdf/Space_Gripper_URDF/bin_stl/finger_lin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
- added link finger_link31_1, mass 0.058758; collision mesh filename=package://fusion2urdf/Space_Gripper_URDF/bin_stl/finger_lin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; visual mesh filename=package://fusion2urdf/Space_Gripper_URDF/bin_stl/finger_lin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
- added link finger_link32_1, mass 0.058758; collision mesh filename=package://fusion2urdf/Space_Gripper_URDF/bin_stl/finger_lin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; visual mesh filename=package://fusion2urdf/Space_Gripper_URDF/bin_stl/finger_lin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
- added link finger_link33_1, mass 0.165174; collision mesh filename=package://fusion2urdf/Space_Gripper_URDF/bin_stl/finger_lin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; visual mesh filename=package://fusion2urdf/Space_Gripper_URDF/bin_stl/finger_lin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
- added link palm_link1_1, mass 0.04512; collision mesh filename=package://fusion2urdf/Space_Gripper_URDF/bin_stl/palm_link1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; visual mesh filename=package://fusion2urdf/Space_Gripper_URDF/bin_stl/palm_link1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
- added link palm_link2_1, mass 0.04512; collision mesh filename=package://fusion2urdf/Space_Gripper_URDF/bin_stl/palm_link2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; visual mesh filename=package://fusion2urdf/Space_Gripper_URDF/bin_stl/palm_link2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
- added link palm_link3_1, mass 0.04512; collision mesh filename=package://fusion2urdf/Space_Gripper_URDF/bin_stl/palm_link3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; visual mesh filename=package://fusion2urdf/Space_Gripper_URDF/bin_stl/palm_link3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
- link base_link: mass 0.1968623967275559 -> 0.196862; geometry collision mesh filename=package://fusion2urdf/Space_Gripper_URDF/bin_stl/base_link_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; visual mesh filename=package://fusion2urdf/Space_Gripper_URDF/bin_stl/base_link_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
Joints:
- joint finger_joint_1_1: axis -0.0 -1.0 0.0 -> -0.0 -0.01 0.0; child finger_link111 -> finger_link11_1; parent palm_link11 -> palm_link1_1
- joint finger_joint_1_2: axis 0.0 1.0 0.0 -> 0.0 0.01 0.0; child finger_link121 -> finger_link12_1; parent finger_link111 -> finger_link11_1
- joint finger_joint_1_3: axis -0.0 -1.0 -0.0 -> 0.0 0.01 0.0; child finger_link131 -> finger_link13_1; limit lower=-1.570796 upper=0.0 effort=100 velocity=100 -> lower=-1.570796 upper=1.570796 effort=100 velocity=100; parent finger_link121 -> finger_link12_1
- joint finger_joint_2_1: axis -0.866025 -0.5 -0.0 -> -0.00866 -0.005 -0.0; child finger_link211 -> finger_link21_1; parent palm_link21 -> palm_link2_1
- joint finger_joint_2_2: axis -0.866025 -0.5 0.0 -> -0.00866 -0.005 0.0; child finger_link221 -> finger_link22_1; parent finger_link211 -> finger_link21_1
- joint finger_joint_2_3: axis -0.866025 -0.5 0.0 -> -0.00866 -0.005 0.0; child finger_link231 -> finger_link23_1; limit lower=0.0 upper=1.570796 effort=100 velocity=100 -> lower=-1.570796 upper=1.570796 effort=100 velocity=100; parent finger_link221 -> finger_link22_1
- joint finger_joint_3_1: axis -0.866025 0.5 0.0 -> -0.00866 0.005 0.0; child finger_link311 -> finger_link31_1; parent palm_link31 -> palm_link3_1
- joint finger_joint_3_2: axis -0.866025 0.5 -0.0 -> -0.00866 0.005 -0.0; child finger_link321 -> finger_link32_1; parent finger_link311 -> finger_link31_1
- joint finger_joint_3_3: axis -0.866025 0.5 -0.0 -> 0.00866 -0.005 0.0; child finger_link331 -> finger_link33_1; limit lower=-1.570796 upper=0.0 effort=100 velocity=100 -> lower=-1.570796 upper=1.570796 effort=100 velocity=100; parent finger_link321 -> finger_link32_1
- joint palm_joint_1: axis -0.0 0.0 1.0 -> -0.0 0.0 0.01; child palm_link11 -> palm_link1_1
- joint palm_joint_2: axis -0.0 0.0 -1.0 -> -0.0 0.0 -0.01; child palm_link31 -> palm_link3_1
- joint palm_joint_3: axis -0.0 -0.0 1.0 -> -0.0 -0.0 0.01; child palm_link21 -> palm_link2_1

Commit message: URDF execution fix

File: Visualization/PyBullet/Space_Gripper_URDF.urdf (robot description, URDF)
Before this commit: robot Space_Gripper_URDF, 13 links, 12 joints
Links:
- removed link finger_link11_1
- removed link finger_link12_1
- removed link finger_link13_1
- removed link finger_link21_1
- removed link finger_link22_1
- removed link finger_link23_1
- removed link finger_link31_1
- removed link finger_link32_1
- removed link finger_link33_1
- removed link palm_link1_1
- removed link palm_link2_1
- removed link palm_link3_1
- added link finger_link111, mass 0.058757815724503226; collision mesh filename=meshes/finger_link111.stl scale=0.001 0.001 0.001; visual mesh filename=meshes/finger_link111.stl scale=0.001 0.001 0.001
- added link finger_link121, mass 0.05875781572450322; collision mesh filename=meshes/finger_link121.stl scale=0.001 0.001 0.001; visual mesh filename=meshes/finger_link121.stl scale=0.001 0.001 0.001
- added link finger_link131, mass 0.16517380192384765; collision mesh filename=meshes/finger_link131.stl scale=0.001 0.001 0.001; visual mesh filename=meshes/finger_link131.stl scale=0.001 0.001 0.001
- added link finger_link211, mass 0.05875781572450313; collision mesh filename=meshes/finger_link211.stl scale=0.001 0.001 0.001; visual mesh filename=meshes/finger_link211.stl scale=0.001 0.001 0.001
- added link finger_link221, mass 0.05875781572450321; collision mesh filename=meshes/finger_link221.stl scale=0.001 0.001 0.001; visual mesh filename=meshes/finger_link221.stl scale=0.001 0.001 0.001
- added link finger_link231, mass 0.1651738019238477; collision mesh filename=meshes/finger_link231.stl scale=0.001 0.001 0.001; visual mesh filename=meshes/finger_link231.stl scale=0.001 0.001 0.001
- added link finger_link311, mass 0.058757815724503115; collision mesh filename=meshes/finger_link311.stl scale=0.001 0.001 0.001; visual mesh filename=meshes/finger_link311.stl scale=0.001 0.001 0.001
- added link finger_link321, mass 0.05875781572450316; collision mesh filename=meshes/finger_link321.stl scale=0.001 0.001 0.001; visual mesh filename=meshes/finger_link321.stl scale=0.001 0.001 0.001
- added link finger_link331, mass 0.16517380192142656; collision mesh filename=meshes/finger_link331.stl scale=0.001 0.001 0.001; visual mesh filename=meshes/finger_link331.stl scale=0.001 0.001 0.001
- added link palm_link11, mass 0.04512002505288437; collision mesh filename=meshes/palm_link11.stl scale=0.001 0.001 0.001; visual mesh filename=meshes/palm_link11.stl scale=0.001 0.001 0.001
- added link palm_link21, mass 0.04512002511118007; collision mesh filename=meshes/palm_link21.stl scale=0.001 0.001 0.001; visual mesh filename=meshes/palm_link21.stl scale=0.001 0.001 0.001
- added link palm_link31, mass 0.04512002511118017; collision mesh filename=meshes/palm_link31.stl scale=0.001 0.001 0.001; visual mesh filename=meshes/palm_link31.stl scale=0.001 0.001 0.001
- link base_link: mass 0.196862 -> 0.19686239672755595; geometry collision mesh filename=meshes/base_link.stl scale=0.001 0.001 0.001; visual mesh filename=meshes/base_link.stl scale=0.001 0.001 0.001
Joints:
- joint finger_joint_1_1: axis -0.0 -0.01 0.0 -> -0.0 -1.0 0.0; child finger_link11_1 -> finger_link111; parent palm_link1_1 -> palm_link11
- joint finger_joint_1_2: axis 0.0 0.01 0.0 -> 0.0 1.0 0.0; child finger_link12_1 -> finger_link121; parent finger_link11_1 -> finger_link111
- joint finger_joint_1_3: axis 0.0 0.01 0.0 -> 0.0 1.0 0.0; child finger_link13_1 -> finger_link131; parent finger_link12_1 -> finger_link121
- joint finger_joint_2_1: axis -0.00866 -0.005 -0.0 -> -0.866025 -0.5 -0.0; child finger_link21_1 -> finger_link211; parent palm_link2_1 -> palm_link21
- joint finger_joint_2_2: axis -0.00866 -0.005 0.0 -> -0.866025 -0.5 0.0; child finger_link22_1 -> finger_link221; parent finger_link21_1 -> finger_link211
- joint finger_joint_2_3: axis -0.00866 -0.005 0.0 -> -0.866025 -0.5 0.0; child finger_link23_1 -> finger_link231; parent finger_link22_1 -> finger_link221
- joint finger_joint_3_1: axis -0.00866 0.005 0.0 -> -0.866025 0.5 0.0; child finger_link31_1 -> finger_link311; parent palm_link3_1 -> palm_link31
- joint finger_joint_3_2: axis -0.00866 0.005 -0.0 -> -0.866025 0.5 -0.0; child finger_link32_1 -> finger_link321; parent finger_link31_1 -> finger_link311
- joint finger_joint_3_3: axis 0.00866 -0.005 0.0 -> 0.866025 -0.5 0.0; child finger_link33_1 -> finger_link331; parent finger_link32_1 -> finger_link321
- joint palm_joint_1: axis -0.0 0.0 0.01 -> -0.0 0.0 1.0; child palm_link1_1 -> palm_link11
- joint palm_joint_2: axis -0.0 0.0 -0.01 -> -0.0 0.0 -1.0; child palm_link3_1 -> palm_link31
- joint palm_joint_3: axis -0.0 -0.0 0.01 -> -0.0 -0.0 1.0; child palm_link2_1 -> palm_link21
