Commit message: updated URDF with end_effector

File: Visualization/C6_mini/URDF.urdf (robot description, URDF)
Before this commit: robot URDF, 13 links, 12 joints
Links:
- link base_link: mass 1.965537963955518 -> 1.9655379639555184
- link finger1_ef1: mass 0.07986065950945902 -> 0.23659461522625636
- link finger2_ef1: mass 0.07986065950945906 -> 0.23659461522625652
- link finger3_ef1: mass 0.07986065950945924 -> 0.23659461522625608
- link finger_link231: mass 0.5923964896980345 -> 0.5898232250623396
- link finger_link331: mass 0.592396483561268 -> 0.5898232192882596
Joints:
- joint finger1_joint1: axis -0.0 1.0 -0.0 -> 0.0 1.0 -0.0
- joint finger2_joint3: limit lower=0.0 upper=1.570796 effort=100 velocity=100 -> lower=-1.570796 upper=1.570796 effort=100 velocity=100
- joint finger3_joint3: limit lower=0.0 upper=1.570796 effort=100 velocity=100 -> lower=-1.570796 upper=1.570796 effort=100 velocity=100
